File: MAX713.kicad_pcb (KiCad board)
At the start: 2 copper layers, 76.2 x 76.2 mm, 67 parts, among them M1 IRFR9024, Q1 CMPTA06, Q2 MMBT2907ALT1, Q3 CMPTA06, Q4 CMPTA06, SW1 SW1, SW2 SW2, SW3 SW3, SW4 SW4, U1 MAX713CSE

Commit message: Add files via upload
Parts:
- removed H1, H2, H3, H4: M3, MountingHole:MountingHole_3.2mm_M3_Pad_Via
- removed REF**: Arduino_UNO_R3_WithMountingHoles, Module:Arduino_UNO_R3_WithMountingHoles
- added A1: Arduino_UNO_R3, Module:Arduino_UNO_R3_WithMountingHoles, F.Cu at (149.7, 119.1)
- C1, C2, C3, C4, C5, C6, D1, D2, D4, L1, M1, Q1, Q2, Q3, Q4, R2, R3, R4, R5, R7, R8, TP1, TP10, TP11, TP12, TP13, TP14, TP15, TP16, TP17, TP18, TP19, TP2, TP20, TP21, TP22, TP3, TP4, TP5, TP6, TP7, TP8, TP9, U1: moved to B.Cu
- D3: footprint LED_SMD:LED_0805_2012Metric -> LED_SMD:LED_1206_3216Metric_ReverseMount_Hole1.8x2.4mm; moved to B.Cu
- moved FID2 115.5 mm to (177.7, 165.0)
- moved JP2 111.1 mm to (184.4, 163.6)
- moved JP1 103.9 mm to (181.9, 159.8)
- moved TP8 97.3 mm to (197.7, 155.1), turned to 180 degrees
- moved R1 96.5 mm to (144.3, 160.8), turned to 0 degrees
- moved CONN1 91.8 mm to (127.5, 151.9), turned to -90 degrees
- moved TP9 90.7 mm to (140.0, 161.9), turned to 180 degrees
- moved D4 88.5 mm to (159.5, 160.8), turned to 180 degrees
- moved D3 87.7 mm to (128.5, 165.1), turned to 0 degrees
- moved TP16 86.9 mm to (196.1, 163.3), turned to 0 degrees
- moved TP17 86.9 mm to (198.6, 163.3), turned to 180 degrees
- moved TP10 85.8 mm to (201.4, 143.3), turned to 180 degrees
- moved Q4 85.6 mm to (134.2, 163.1), turned to 180 degrees
- moved C5 85.4 mm to (137.2, 154.4), turned to 90 degrees
- moved TP3 84.1 mm to (194.1, 160.7), turned to 180 degrees
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Routing:
- net /V+: track 146.2 -> 0.00 mm
- net /BATT-: track 96.9 -> 0.00 mm, vias 2 -> 0
- net /REF: track 77.0 -> 0.00 mm, vias 2 -> 0
- net /DRV: track 70.0 -> 0.00 mm, vias 2 -> 0
- net /PGM2: track 54.4 -> 0.00 mm, vias 2 -> 0
- net /PGM3: track 47.4 -> 0.00 mm
- net Net-(Q4-E): track 46.4 -> 0.00 mm, vias 2 -> 0
- net /BATT+: track 41.1 -> 0.00 mm
- net Net-(Q1-B): track 39.8 -> 0.00 mm
- net /PGM0: track 36.5 -> 0.00 mm
- net Net-(Q3-E): track 29.5 -> 0.00 mm, vias 2 -> 0
- net Net-(M1-G): track 29.0 -> 0.00 mm
- net Net-(Q3-B): track 28.1 -> 0.00 mm
- net /PGM1: track 27.8 -> 0.00 mm
- net /LED: track 16.8 -> 0.00 mm
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- removed copper zone on F.Cu, net /BATT+
- removed copper zone on F.Cu, net /BATT-
- removed copper zone on F.Cu, net /VIN
- removed copper zone on B.Cu, net GND
- removed copper zone on F.Cu, net GND
- removed copper zone on F.Cu, net Net-(D1-A)
- removed copper zone on F.Cu, net Net-(D2-K)
Other:
- board size 76.2 x 76.2 mm -> 69.1 x 53.8 mm
- board text added: "${COMPANY} ${COMMENT4}"
- board text added: "+ BATT -"
- board text added: "0"
- board text added: "0 mils"
- board text added: "0.02"
- board text added: "0.3937 mils"
- board text added: "1.37795 mils"
- board text added: "11.81 mils"
- board text added: "2720.00 mils x 2120.00 mils"
- board text added: "3.3"
- board text added: "4.5"
- board text added: "59.44882 mils"
- board text added: "62.99 mils"
- board text added: "7.87 mils / 0.00 mils"
- board text added: "B.Cu"
- board text added: "B.Mask"
- board text added: "B.Paste"
- board text added: "B.Silkscreen"
- board text added: "BOARD CHARACTERISTICS"
- board text added: "Board Thickness:"
- board text added: "Board overall dimensions:"
- board text added: "Bottom Silk Screen"
- board text added: "Bottom Solder Mask"
- board text added: "Bottom Solder Paste"
- board text added: "Castellated pads:"
- board text added: "Color"
- board text added: "Copper Finish:"
- board text added: "Copper Layer Count:"
- board text added: "Dielectric 1"
- board text added: "Direct Printing"
- board text added: "Dry Film"
- board text added: "Edge card connectors:"
- board text added: "Epsilon R"
- board text added: "F.Cu"
- board text added: "F.Mask"
- board text added: "F.Paste"
- board text added: "F.Silkscreen"
- board text added: "FR4"
- board text added: "FR4 natural"
- board text added: "Green"
- board text added: "Impedance Control:"
- board text added: "Layer Name"
- board text added: "Loss Tangent"
- board text added: "Material"
- board text added: "Min hole diameter:"
- board text added: "Min track/spacing:"
- board text added: "No"
- board text added: "None"
- board text added: "Plated Board Edge:"
- board text added: "Thickness (mils)"
- board text added: "Top Silk Screen"
- board text added: "Top Solder Mask"
- board text added: "Top Solder Paste"
- board text added: "Type"
- board text added: "White"
- board text added: "copper"
- board text added: "core"
- board text removed: "- BATT +"
- board text removed: "astroelectronic@ AE01012713"
