File: MAX713.kicad_sch (KiCad schematic)
At the start: 72 parts, among them M1 IRFR9024, Q1 CMPTA06, Q2 MMBT2907ALT1, Q3 CMPTA06, Q4 CMPTA06, SW1 SW1, SW2 SW2, SW3 SW3, SW4 SW4, U1 MAX713CSE

Commit message: Add files via upload
Parts:
- removed H1, H2, H3, H4: M3, MountingHole:MountingHole_3.2mm_M3_Pad_Via, symbol MAX713:MountingHole
- added A1: Arduino_UNO_R3, Module:Arduino_UNO_R3_WithMountingHoles, symbol MCU_Module:Arduino_UNO_R3
- D3: footprint LED_SMD:LED_0805_2012Metric -> LED_SMD:LED_1206_3216Metric_ReverseMount_Hole1.8x2.4mm
Connections:
- net GND: now also A1.29 (GND), A1.6 (GND), A1.7 (GND)
Other:
- moved on the sheet: LOGO1, LOGO2, LOGO3, LOGO4
